Commit message: Fix wrong namespace for the panda hand

File: robots/hand.xacro (robot description, xacro)
@@ -1,13 +1,13 @@
 <?xml version="1.0" encoding="utf-8"?>
 <robot xmlns:xacro="http://www.ros.org/wiki/xacro" name="hand">
-  <xacro:macro name="hand" params="connected_to:='' ns:='' rpy:='0 0 0' xyz:='0 0 0' ">
+  <xacro:macro name="hand" params="connected_to:='' robot_name='' rpy:='0 0 0' xyz:='0 0 0' ">
     <xacro:unless value="${connected_to == ''}">
-      <joint name="${ns}_hand_joint" type="fixed">
+      <joint name="${robot_name}_hand_joint" type="fixed">
         <parent link="${connected_to}"/>
-        <child link="${ns}_hand"/>
+        <child link="${robot_name}_hand"/>
         <origin xyz="${xyz}" rpy="${rpy}"/>
       </joint>
     </xacro:unless>
-    <link name="${ns}_hand">
+    <link name="${robot_name}_hand">
       <visual>
         <geometry>
@@ -26,5 +26,5 @@
       </inertial>
     </link>
-    <link name="${ns}_leftfinger">
+    <link name="${robot_name}_leftfinger">
       <visual>
         <geometry>
@@ -43,5 +43,5 @@
       </inertial>
     </link>
-    <link name="${ns}_rightfinger">
+    <link name="${robot_name}_rightfinger">
       <visual>
         <origin xyz="0 0 0" rpy="0 0 ${pi}"/>
@@ -62,18 +62,18 @@
       </inertial>
     </link>
-    <joint name="${ns}_finger_joint1" type="prismatic">
-      <parent link="${ns}_hand"/>
-      <child link="${ns}_leftfinger"/>
+    <joint name="${robot_name}_finger_joint1" type="prismatic">
+      <parent link="${robot_name}_hand"/>
+      <child link="${robot_name}_leftfinger"/>
       <origin xyz="0 0 0.0584" rpy="0 0 0"/>
       <axis xyz="0 1 0"/>
       <limit effort="20" lower="0.0" upper="0.04" velocity="0.2"/>
     </joint>
-    <joint name="${ns}_finger_joint2" type="prismatic">
-      <parent link="${ns}_hand"/>
-      <child link="${ns}_rightfinger"/>
+    <joint name="${robot_name}_finger_joint2" type="prismatic">
+      <parent link="${robot_name}_hand"/>
+      <child link="${robot_name}_rightfinger"/>
       <origin xyz="0 0 0.0584" rpy="0 0 0"/>
       <axis xyz="0 -1 0"/>
       <limit effort="20" lower="0.0" upper="0.04" velocity="0.2"/>
-      <mimic joint="${ns}_finger_joint1" />
+      <mimic joint="${robot_name}_finger_joint1" />
     </joint>
   </xacro:macro>

File: robots/panda_arm_world.urdf.xacro (robot description, xacro)
@@ -6,5 +6,5 @@
   <xacro:panda_arm />
   <xacro:include filename="$(find easy_panda_sim)/robots/hand.xacro"/>
-  <xacro:hand rpy="0 0 ${-pi/4}" connected_to="panda_link8"/>
+  <xacro:hand rpy="0 0 ${-pi/4}" robot_name="$(arg robot_name)" connected_to="panda_link8"/>
   <xacro:include filename="$(find easy_panda_sim)/robots/panda.gazebo.xacro"/>
   <xacro:panda_gazebo robot_name="$(arg robot_name)" />

Commit message: Add default tool center point link and associated joint to robots/hand.xacro

File: robots/hand.xacro (robot description, xacro)
@@ -62,4 +62,6 @@
       </inertial>
     </link>
+    <link name="${robot_name}_tcp">
+    </link>
     <joint name="${robot_name}_finger_joint1" type="prismatic">
       <parent link="${robot_name}_hand"/>
@@ -77,4 +79,10 @@
       <mimic joint="${robot_name}_finger_joint1" />
     </joint>
+    <joint name="${robot_name}_tcp_joint" type="fixed">
+      <parent link="${robot_name}_hand"/>
+      <child link="${robot_name}_tcp"/>
+      <origin xyz="0 0 0.12" rpy="0 0 0"/>
+      <axis xyz="0 -1 0"/>
+    </joint>
   </xacro:macro>
 </robot>
