Commit message: Fix type of joint panda_joint8

File: robots/panda_arm.xacro (robot description, xacro)
@@ -249,5 +249,5 @@
       </inertial>
     </link>
-    <joint name="${arm_id}_joint8" type="revolute">
+    <joint name="${arm_id}_joint8" type="fixed">
       <origin rpy="0 0 0" xyz="0 0 0.107"/>
       <parent link="${arm_id}_link7"/>
