Commit message: Add transimissions for panda fingers

File: robots/panda.transmission.xacro (robot description, xacro)
@@ -87,4 +87,24 @@
             </actuator>
         </transmission>
+        <transmission name="${robot_name}_tran_9">
+            <type>transmission_interface/SimpleTransmission</type>
+            <joint name="${robot_name}_finger_joint1">
+                <hardwareInterface>hardware_interface/PositionJointInterface</hardwareInterface>
+            </joint>
+            <actuator name="${robot_name}_motor_9">
+                <hardwareInterface>hardware_interface/PositionJointInterface</hardwareInterface>
+                <mechanicalReduction>1</mechanicalReduction>
+            </actuator>
+        </transmission>
+        <transmission name="${robot_name}_tran_10">
+            <type>transmission_interface/SimpleTransmission</type>
+            <joint name="${robot_name}_finger_joint2">
+                <hardwareInterface>hardware_interface/PositionJointInterface</hardwareInterface>
+            </joint>
+            <actuator name="${robot_name}_motor_10">
+                <hardwareInterface>hardware_interface/PositionJointInterface</hardwareInterface>
+                <mechanicalReduction>1</mechanicalReduction>
+            </actuator>
+        </transmission>
     </xacro:macro>
 </robot>

Commit message: Fix wrong Gazebo transmission configuration

File: robots/panda.transmission.xacro (robot description, xacro)
@@ -79,5 +79,5 @@
         <transmission name="${robot_name}_tran_8">
             <type>transmission_interface/SimpleTransmission</type>
-            <joint name="${robot_name}_joint8">
+            <joint name="${robot_name}_finger_joint1">
                 <hardwareInterface>hardware_interface/PositionJointInterface</hardwareInterface>
             </joint>
@@ -89,5 +89,5 @@
         <transmission name="${robot_name}_tran_9">
             <type>transmission_interface/SimpleTransmission</type>
-            <joint name="${robot_name}_finger_joint1">
+            <joint name="${robot_name}_finger_joint2">
                 <hardwareInterface>hardware_interface/PositionJointInterface</hardwareInterface>
             </joint>
@@ -97,14 +97,4 @@
             </actuator>
         </transmission>
-        <transmission name="${robot_name}_tran_10">
-            <type>transmission_interface/SimpleTransmission</type>
-            <joint name="${robot_name}_finger_joint2">
-                <hardwareInterface>hardware_interface/PositionJointInterface</hardwareInterface>
-            </joint>
-            <actuator name="${robot_name}_motor_10">
-                <hardwareInterface>hardware_interface/PositionJointInterface</hardwareInterface>
-                <mechanicalReduction>1</mechanicalReduction>
-            </actuator>
-        </transmission>
     </xacro:macro>
 </robot>
